Commit message: Add working version

File: RHexGym/rsc/urdf/RHex.urdf (robot description, URDF)
Before this commit: robot RHex, 13 links, 12 joints
Links:
- link link_body: geometry collision box size=0.50 0.23 0.10; visual mesh filename=../meshes/rhex_body.dae scale=1.0 1.0 1.0
- link link_leg1Lower: geometry collision sphere radius=0.0050; collision sphere radius=0.0075
- link link_leg1Upper: geometry collision sphere radius=0.0075; collision sphere radius=0.0075
- link link_leg2Lower: geometry collision sphere radius=0.0050; collision sphere radius=0.0075
- link link_leg2Upper: geometry collision sphere radius=0.0075; collision sphere radius=0.0075
- link link_leg3Lower: geometry collision sphere radius=0.0050; collision sphere radius=0.0075
- link link_leg3Upper: geometry collision sphere radius=0.0075; collision sphere radius=0.0075
- link link_leg4Lower: geometry collision sphere radius=0.0050; collision sphere radius=0.0075
- link link_leg4Upper: geometry collision sphere radius=0.0075; collision sphere radius=0.0075
- link link_leg5Lower: geometry collision sphere radius=0.0050; collision sphere radius=0.0075
- link link_leg5Upper: geometry collision sphere radius=0.0075; collision sphere radius=0.0075
- link link_leg6Lower: geometry collision sphere radius=0.0050; collision sphere radius=0.0075
- link link_leg6Upper: geometry collision sphere radius=0.0075; collision sphere radius=0.0075
Joints:
- removed joint joint1
- removed joint joint2
- removed joint joint3
- removed joint joint4
- removed joint joint5
- removed joint joint6
- added joint hip_joint1: type revolute, parent link_body, child link_leg1Upper, origin xyz=0.25 0.15 0 rpy=0 0 0, axis 0 -1 0, limit effort=20 velocity=25
- added joint hip_joint2: type revolute, parent link_body, child link_leg2Upper, origin xyz=0 0.20 0 rpy=0 0 0, axis 0 -1 0, limit effort=20 velocity=25
- added joint hip_joint3: type revolute, parent link_body, child link_leg3Upper, origin xyz=-0.25 0.15 0 rpy=0 0 0, axis 0 -1 0, limit effort=20 velocity=25
- added joint hip_joint4: type revolute, parent link_body, child link_leg4Upper, origin xyz=-0.25 -0.15 0 rpy=0 0 0, axis 0 -1 0, limit effort=20 velocity=25
- added joint hip_joint5: type revolute, parent link_body, child link_leg5Upper, origin xyz=0 -0.20 0 rpy=0 0 0, axis 0 -1 0, limit effort=20 velocity=25
- added joint hip_joint6: type revolute, parent link_body, child link_leg6Upper, origin xyz=0.25 -0.15 0 rpy=0 0 0, axis 0 -1 0, limit effort=20 velocity=25
- joint Leg1Joint: origin xyz=-0.080 0.0 -0.099 rpy=0 0 0 -> xyz=-0.080 0.0 -0.095 rpy=0 0 0
- joint Leg2Joint: origin xyz=-0.080 0.0 -0.099 rpy=0 0 0 -> xyz=-0.080 0.0 -0.095 rpy=0 0 0
- joint Leg3Joint: origin xyz=-0.080 0.0 -0.099 rpy=0 0 0 -> xyz=-0.080 0.0 -0.095 rpy=0 0 0
- joint Leg4Joint: origin xyz=-0.080 0.0 -0.099 rpy=0 0 0 -> xyz=-0.080 0.0 -0.095 rpy=0 0 0
- joint Leg5Joint: origin xyz=-0.080 0.0 -0.099 rpy=0 0 0 -> xyz=-0.080 0.0 -0.095 rpy=0 0 0
- joint Leg6Joint: origin xyz=-0.080 0.0 -0.099 rpy=0 0 0 -> xyz=-0.080 0.0 -0.095 rpy=0 0 0
